File: 2.3 Circuit Diagram/Inoovatest/MCU_and_display.kicad_sch (KiCad schematic)
At the start: 6 parts, among them J6 USB_A, Q10 AO3400A, U18 TouchScreen/SPI Touch Control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

Commit message: more datasheets
Parts:
- renumbered R56 to R55, R57 to R56, U19 to U18, U18 to U19
Connections:
- net at U19.4 (NC): now also U18.14 (GPIO13/ADC)
Changed lines of the file:
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@@
 		(on_board yes)
 		(dnp no)
-		(property "Reference" "#PWR0174"
+		(property "Reference" "#PWR0158"
 			(at 252.222 178.308 0)
 			(effects
@@
 			(project "Inoovatest"
 				(path "/e09d161e-639f-4600-8aa9-665b6b461114/ce96d435-3607-40fc-9966-258a09df953a"
-					(reference "#PWR0174")
+					(reference "#PWR0158")
 					(unit 1)
 				)
@@
 		(on_board yes)
 		(dnp no)
-		(property "Reference" "#PWR0180"
+		(property "Reference" "#PWR0151"
 			(at 291.846 96.012 0)
 			(effects
@@
 			(project "Inoovatest"
 				(path "/e09d161e-639f-4600-8aa9-665b6b461114/ce96d435-3607-40fc-9966-258a09df953a"
-					(reference "#PWR0180")
+					(reference "#PWR0151")
 					(unit 1)
 				)
@@
 		(dnp no)
 		(fields_autoplaced yes)
-		(property "Reference" "#PWR0170"
+		(property "Reference" "#PWR0147"
 			(at 223.012 83.566 0)
 			(effects
@@
 			(project "Inoovatest"
 				(path "/e09d161e-639f-4600-8aa9-665b6b461114/ce96d435-3607-40fc-9966-258a09df953a"
-					(reference "#PWR0170")
+					(reference "#PWR0147")
 					(unit 1)
 				)
@@
 		(on_board yes)
 		(dnp no)
-		(property "Reference" "#PWR0178"
+		(property "Reference" "#PWR0150"
 			(at 287.02 92.202 0)
 			(effects
@@
 			(project "Inoovatest"
 				(path "/e09d161e-639f-4600-8aa9-665b6b461114/ce96d435-3607-40fc-9966-258a09df953a"
-					(reference "#PWR0178")
+					(reference "#PWR0150")
 					(unit 1)
 				)
@@
 		(on_board yes)
 		(dnp no)
-		(property "Reference" "#PWR0177"
+		(property "Reference" "#PWR0149"
 			(at 282.702 88.392 0)
 			(effects
@@
 			(project "Inoovatest"
 				(path "/e09d161e-639f-4600-8aa9-665b6b461114/ce96d435-3607-40fc-9966-258a09df953a"
-					(reference "#PWR0177")
+					(reference "#PWR0149")
 					(unit 1)
 				)
@@
 		(on_board yes)
 		(dnp no)
-		(property "Reference" "R56"
+		(property "Reference" "R55"
 			(at 148.082 149.352 90)
 			(effects
@@
 			(project "Inoovatest"
 				(path "/e09d161e-639f-4600-8aa9-665b6b461114/ce96d435-3607-40fc-9966-258a09df953a"
-					(reference "R56")
+					(reference "R55")
 					(unit 1)
 				)
@@
 		(on_board yes)
 		(dnp no)
-		(property "Reference" "#PWR0173"
+		(property "Reference" "#PWR0160"
 			(at 250.444 189.738 0)
 			(effects
@@
 			(project "Inoovatest"
 				(path "/e09d161e-639f-4600-8aa9-665b6b461114/ce96d435-3607-40fc-9966-258a09df953a"
-					(reference "#PWR0173")
+					(reference "#PWR0160")
 					(unit 1)
 				)
@@
 		(on_board yes)
 		(dnp no)
-		(property "Reference" "#PWR0175"
+		(property "Reference" "#PWR0163"
 			(at 260.604 214.884 0)
 			(effects
@@
 			(project "Inoovatest"
 				(path "/e09d161e-639f-4600-8aa9-665b6b461114/ce96d435-3607-40fc-9966-258a09df953a"
-					(reference "#PWR0175")
+					(reference "#PWR0163")
 					(unit 1)
 				)
@@
 		(on_board yes)
 		(dnp no)
-		(property "Reference" "#PWR0169"
+		(property "Reference" "#PWR0161"
 			(at 207.01 194.564 0)
 			(effects
@@
 			(project "Inoovatest"
 				(path "/e09d161e-639f-4600-8aa9-665b6b461114/ce96d435-3607-40fc-9966-258a09df953a"
-					(reference "#PWR0169")
+					(reference "#PWR0161")
 					(unit 1)
 				)
@@
 		(on_board yes)
 		(dnp no)
-		(property "Reference" "#PWR0164"
+		(property "Reference" "#PWR0155"
 			(at 143.764 148.082 0)
 			(effects
@@
 			(project "Inoovatest"
 				(path "/e09d161e-639f-4600-8aa9-665b6b461114/ce96d435-3607-40fc-9966-258a09df953a"
-					(reference "#PWR0164")
+					(reference "#PWR0155")
 					(unit 1)
 				)
@@
 		(on_board yes)
 		(dnp no)
-		(property "Reference" "#PWR0157"
+		(property "Reference" "#PWR0154"
 			(at 96.774 125.222 0)
 			(effects
@@
 			(project "Inoovatest"
 				(path "/e09d161e-639f-4600-8aa9-665b6b461114/ce96d435-3607-40fc-9966-258a09df953a"
-					(reference "#PWR0157")
+					(reference "#PWR0154")
 					(unit 1)
 				)
@@
 		(dnp no)
 		(fields_autoplaced yes)
-		(property "Reference" "#PWR0168"
+		(property "Reference" "#PWR0146"
 			(at 192.532 83.312 0)
 			(effects
@@
 			(project "Inoovatest"
 				(path "/e09d161e-639f-4600-8aa9-665b6b461114/ce96d435-3607-40fc-9966-258a09df953a"
-					(reference "#PWR0168")
+					(reference "#PWR0146")
 					(unit 1)
 				)
@@
 		(on_board yes)
 		(dnp no)
-		(property "Reference" "#PWR0179"
+		(property "Reference" "#PWR0153"
 			(at 289.052 120.904 0)
 			(effects
@@
 			(project "Inoovatest"
 				(path "/e09d161e-639f-4600-8aa9-665b6b461114/ce96d435-3607-40fc-9966-258a09df953a"
-					(reference "#PWR0179")
+					(reference "#PWR0153")
 					(unit 1)
 				)
@@
 		(on_board yes)
 		(dnp no)
-		(property "Reference" "U18"
+		(property "Reference" "U19"
 			(at 146.558 181.356 0)
 			(effects
@@
 			(project "Inoovatest"
 				(path "/e09d161e-639f-4600-8aa9-665b6b461114/ce96d435-3607-40fc-9966-258a09df953a"
-					(reference "U18")
+					(reference "U19")
 					(unit 1)
 				)
@@
 		(on_board yes)
 		(dnp no)
-		(property "Reference" "#PWR0166"
+		(property "Reference" "#PWR0159"
 			(at 172.974 184.912 0)
 			(effects
@@
 			(project "Inoovatest"
 				(path "/e09d161e-639f-4600-8aa9-665b6b461114/ce96d435-3607-40fc-9966-258a09df953a"
-					(reference "#PWR0166")
+					(reference "#PWR0159")
 					(unit 1)
 				)
@@
 		(on_board yes)
 		(dnp no)
-		(property "Reference" "R57"
+		(property "Reference" "R56"
 			(at 148.082 146.812 90)
 			(effects
@@
 			(project "Inoovatest"
 				(path "/e09d161e-639f-4600-8aa9-665b6b461114/ce96d435-3607-40fc-9966-258a09df953a"
-					(reference "R57")
+					(reference "R56")
 					(unit 1)
 				)
@@
 		(on_board yes)
 		(dnp no)
-		(property "Reference" "#PWR0165"
+		(property "Reference" "#PWR0156"
 			(at 158.75 165.608 0)
 			(effects
@@
 			(project "Inoovatest"
 				(path "/e09d161e-639f-4600-8aa9-665b6b461114/ce96d435-3607-40fc-9966-258a09df953a"
-					(reference "#PWR0165")
+					(reference "#PWR0156")
 					(unit 1)
 				)
@@
 		(on_board yes)
 		(dnp no)
-		(property "Reference" "#PWR0167"
+		(property "Reference" "#PWR0164"
 			(at 173.228 229.616 0)
 			(effects
@@
 			(project "Inoovatest"
 				(path "/e09d161e-639f-4600-8aa9-665b6b461114/ce96d435-3607-40fc-9966-258a09df953a"
-					(reference "#PWR0167")
+					(reference "#PWR0164")
 					(unit 1)
 				)
@@
 		(on_board yes)
 		(dnp no)
-		(property "Reference" "#PWR0171"
+		(property "Reference" "#PWR0162"
 			(at 232.156 211.074 0)
 			(effects
@@
 			(project "Inoovatest"
 				(path "/e09d161e-639f-4600-8aa9-665b6b461114/ce96d435-3607-40fc-9966-258a09df953a"
-					(reference "#PWR0171")
+					(reference "#PWR0162")
 					(unit 1)
 				)
@@
 		(dnp no)
 		(fields_autoplaced yes)
-		(property "Reference" "#PWR0172"
+		(property "Reference" "#PWR0148"
 			(at 238.252 83.566 0)
 			(effects
@@
 			(project "Inoovatest"
 				(path "/e09d161e-639f-4600-8aa9-665b6b461114/ce96d435-3607-40fc-9966-258a09df953a"
-					(reference "#PWR0172")
+					(reference "#PWR0148")
 					(unit 1)
 				)
@@
 		(on_board yes)
 		(dnp no)
-		(property "Reference" "#PWR0181"
+		(property "Reference" "#PWR0152"
 			(at 296.418 99.568 0)
 			(effects
@@
 			(project "Inoovatest"
 				(path "/e09d161e-639f-4600-8aa9-665b6b461114/ce96d435-3607-40fc-9966-258a09df953a"
-					(reference "#PWR0181")
+					(reference "#PWR0152")
 					(unit 1)
 				)
@@
 		(on_board yes)
 		(dnp no)
-		(property "Reference" "#PWR0176"
+		(property "Reference" "#PWR0157"
 			(at 272.034 177.8 0)
 			(effects
@@
 			(project "Inoovatest"
 				(path "/e09d161e-639f-4600-8aa9-665b6b461114/ce96d435-3607-40fc-9966-258a09df953a"
-					(reference "#PWR0176")
+					(reference "#PWR0157")
 					(unit 1)
 				)
@@
 		(on_board yes)
 		(dnp no)
-		(property "Reference" "U19"
+		(property "Reference" "U18"
 			(at 263.906 82.042 0)
 			(effects
@@
 			(project "Inoovatest"
 				(path "/e09d161e-639f-4600-8aa9-665b6b461114/ce96d435-3607-40fc-9966-258a09df953a"
-					(reference "U19")
-					(unit 1)
-				)
+					(reference "U18")
+					(unit 1)
+				)
