File: 2.3 Circuit Diagram/Inoovatest/power-regulation.kicad_sch (KiCad schematic)
At the start: 28 parts, among them U1 TPS61170, U10 TPS61089, U3 TPS61099

Commit message: more datasheets
Parts:
- renumbered Buck_Convertor1 to Buck_Convertor2, C27 to C39, C23 to C40, C25 to C41, C8 to C42, C11 to C43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
