File: 2.3 Circuit Diagram/Inoovatest_Main/MCU_and_display.kicad_sch (KiCad schematic)
At the start: 11 parts, among them J6 USB_A, Q7 AO3400A, SW4 Emergency Stop, U19 W25Q128JVS, U22 TouchScreen/SPI Touch Control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

Commit message: 3D Models for electrical parts
- added all the 3D models for ports
- created necessary footprints
Parts:
- renumbered C77 to C75, C78 to C76, Q7 to Q12, R58 to R70, R59 to R71, R60 to R72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
