File: 2.3 Circuit Diagram/Inoovatest_Subsystems/Inoovatest_Sub.kicad_pcb (KiCad board)
At the start: 2 copper layers, 120 x 100 mm, 115 parts, among them IC1 MCP73223, IC2 MAX6126, J1 M12 5-pin, J2 USB_A, J3 USB_C Charging port, Q1 AO3401A, Q2 AO3401A, Q3 AO3400A, Q4 AO3400A, Q5 AO3401A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

Commit message: PCB Assembly
Parts:
- moved H3 3.64 mm to (70.0, 46.5)
- moved H1 3.00 mm to (173.0, 30.0)
- moved H4 2.83 mm to (70.0, 113.0)
- moved H2 1.00 mm to (77.0, 30.0)
Changed lines of the file:
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@@
 		(tenting front back)
 		(pcbplotparams
-			(layerselection 0x00000000_00000000_55555555_5755f5ff)
+			(layerselection 0x00000000_00000000_55555555_55555554)
 			(plot_on_all_layers_selection 0x00000000_00000000_00000000_00000000)
 			(disableapertmacros no)
@@
 			(psnegative no)
 			(psa4output no)
-			(plot_black_and_white yes)
+			(plot_black_and_white no)
 			(sketchpadsonfab no)
 			(plotpadnumbers no)
@@
 			(crossoutdnponfab yes)
 			(subtractmaskfromsilk no)
-			(outputformat 1)
+			(outputformat 4)
 			(mirror no)
-			(drillshape 1)
+			(drillshape 0)
 			(scaleselection 1)
 			(outputdirectory "")
@@
 	(footprint "MountingHole:MountingHole_2.2mm_M2_DIN965"
 		(layer "F.Cu")
-		(at 76 30)
+		(at 77 30)
 		(descr "Mounting Hole 2.2mm, M2, no annular, generated by kicad-footprint-generator mountinghole.py")
 		(tags "mountinghole M2 DIN965")
@@
 	(footprint "MountingHole:MountingHole_2.2mm_M2_DIN965"
 		(layer "F.Cu")
-		(at 71 50)
+		(at 70 46.5)
 		(descr "Mounting Hole 2.2mm, M2, no annular, generated by kicad-footprint-generator mountinghole.py")
 		(tags "mountinghole M2 DIN965")
@@
 	(footprint "MountingHole:MountingHole_2.2mm_M2_DIN965"
 		(layer "F.Cu")
-		(at 170 30)
+		(at 173 30)
 		(descr "Mounting Hole 2.2mm, M2, no annular, generated by kicad-footprint-generator mountinghole.py")
 		(tags "mountinghole M2 DIN965")
@@
 	(footprint "MountingHole:MountingHole_2.2mm_M2_DIN965"
 		(layer "F.Cu")
-		(at 72 111)
+		(at 70 113)
 		(descr "Mounting Hole 2.2mm, M2, no annular, generated by kicad-footprint-generator mountinghole.py")
 		(tags "mountinghole M2 DIN965")
@@
 		)
 		(pad "" np_thru_hole circle
-			(at -5.73 -5.77)
+			(at -6.77 -5.79)
 			(size 2.8 2.8)
 			(drill 2.8)
@@
 		)
 		(pad "" np_thru_hole circle
-			(at 9.27 -5.77)
-			(size 2.8 2.8)
-			(drill 2.8)
-			(layers "*.Cu" "*.Mask")
-		)
-		(pad "" np_thru_hole circle
 			(at 9.27 -1.77)
 			(size 2.05 2.05)
@@
 			(layers "*.Cu" "*.Mask")
 		)
+		(pad "" np_thru_hole circle
+			(at 10.25 -5.79)
+			(size 2.8 2.8)
+			(drill 2.8)
+			(layers "*.Cu" "*.Mask")
+		)
 		(pad "1" thru_hole circle
 			(at 0 -3.5)
@@
 	)
 	(gr_rect
+		(start 65 25)
+		(end 70 46.5)
+		(stroke
+			(width 0.1)
+			(type default)
+		)
+		(fill no)
+		(layer "Dwgs.User")
+	)
+	(gr_rect
 		(start 89.05 39.05)
 		(end 134.05 72.55)
@@
 	)
 	(gr_rect
+		(start 173 25)
+		(end 185 30)
+		(stroke
+			(width 0.1)
+			(type default)
+		)
+		(fill no)
+		(layer "Dwgs.User")
+	)
+	(gr_rect
 		(start 65 25)
 		(end 89.05 39.05)
 		(stroke
 			(width 0.1)
+			(type default)
+		)
+		(fill no)
+		(layer "Dwgs.User")
+	)
+	(gr_rect
+		(start 65 113)
+		(end 70 125)
+		(stroke
+			(width 0.1)
+			(type default)
+		)
+		(fill no)
+		(layer "Dwgs.User")
+	)
+	(gr_rect
+		(start 65 25)
+		(end 77 30)
+		(stroke
+			(width 0.1)
