File: 2.3 Circuit Diagram/M12_Connector/M12_Connector.kicad_sch (KiCad schematic)
At the start: 0 parts

Commit message: gggg
Parts:
- added J1: Conn_01x05, symbol Connector_Generic:Conn_01x05
- added R1: 100kΩ, symbol Device:R
- added R2: R, symbol Device:R
Connections:
- new net GND: J1.5 (Pin_5), R2.2
- new net ID: J1.4 (Pin_4), R1.2, R2.1
- new net S+: J1.2 (Pin_2)
- new net S-: J1.3 (Pin_3)
- new net VCC: J1.1 (Pin_1), R1.1
